File: DevboardPCB/DevboardPCB.kicad_sch (KiCad schematic)
At the start: 32 parts, among them J1 USB_C_Receptacle_USB2.0_14P, J2 Conn_01x20, J3 Conn_01x20, J4 Conn_01x03, SW1 SW_Push, U1 RP2040, U2 NCP1117-3.3_SOT223, U3 W25Q128JVS, Y1 12 MHz

Commit message: finished routing
Parts:
- removed U2: NCP1117-3.3_SOT223, Package_TO_SOT_SMD:SOT-223-3_TabPin2, symbol Regulator_Linear:NCP1117-3.3_SOT223
- added C17: 0.1uF, Capacitor_SMD:C_0402_1005Metric, symbol Device:C
- added J10, J12, J7, J8: Conn_01x08, Connector_PinHeader_2.54mm:PinHeader_1x08_P2.54mm_Vertical, symbol Connector_Generic:Conn_01x08
- added J11, J5, J6, J9: Conn_01x02, Connector_PinHeader_2.54mm:PinHeader_1x02_P2.54mm_Vertical, symbol Connector_Generic:Conn_01x02
- added U4: MCP1700x-330xxTT, Package_TO_SOT_SMD:SOT-23, symbol Regulator_Linear:MCP1700x-330xxTT
- C1, C10, C11, C12, C2, C3, C4, C5, C6, C7, C8, C9: footprint (none) -> Capacitor_SMD:C_0402_1005Metric
- C13, C14: footprint (none) -> Capacitor_SMD:C_0603_1608Metric
- C15, C16: value 15pF -> 33pF; footprint (none) -> Capacitor_SMD:C_0402_1005Metric
- J1: footprint (none) -> Connector_USB:USB_C_Receptacle_HRO_TYPE-C-31-M-12
- J2, J3: footprint (none) -> Connector_PinHeader_2.54mm:PinHeader_1x20_P2.54mm_Vertical
- J4: footprint (none) -> Connector_PinHeader_2.54mm:PinHeader_1x03_P2.54mm_Vertical
- R1, R2, R3, R4, R5, R6, R7: footprint (none) -> Resistor_SMD:R_0402_1005Metric
- SW1: footprint (none) -> Button_Switch_SMD:SW_Push_SPST_NO_Alps_SKRK
- U3: value W25Q128JVS -> W25Q16JVZPIQ TR; footprint Package_SO:SOIC-8_5.23x5.23mm_P1.27mm -> Package_SON:Winbond_USON-8-1EP_3x2mm_P0.5mm_EP0.2x1.6mm
- Y1: footprint (none) -> Crystal:Crystal_SMD_3225-4Pin_3.2x2.5mm
Connections:
- net +3V3: now also C17.1, J10.2 (Pin_2), J7.2 (Pin_2), U4.2 (VO)
- net GND: now also C17.2, J10.3 (Pin_3), J10.8 (Pin_8), J12.8 (Pin_8), J7.3 (Pin_3), J7.8 (Pin_8), J8.8 (Pin_8), U4.1 (GND)
- net GPIO0: now also J8.1 (Pin_1)
- net GPIO1: now also J8.7 (Pin_7)
- net GPIO16: now also J12.2 (Pin_2)
- net GPIO17: now also J12.3 (Pin_3)
- net GPIO18: now also J12.5 (Pin_5)
- net GPIO19: now also J12.6 (Pin_6)
- net GPIO2: now also J12.1 (Pin_1)
- net GPIO20: now also J12.4 (Pin_4)
- net GPIO3: now also J12.7 (Pin_7)
- net GPIO4: now also J8.2 (Pin_2)
- net GPIO5: now also J8.3 (Pin_3)
- net GPIO6: now also J8.5 (Pin_5)
- net GPIO7: now also J8.6 (Pin_6)
- net GPIO8: now also J8.4 (Pin_4)
- net USB_D+: now also J10.1 (Pin_1), J7.1 (Pin_1)
- net VBUS: now also U4.3 (VI)
- new net: J10.7 (Pin_7), J9.1 (Pin_1)
- new net: J10.6 (Pin_6), J9.2 (Pin_2)
- new net: J5.2 (Pin_2), J7.4 (Pin_4)
- new net: J5.1 (Pin_1), J7.5 (Pin_5)
- new net: J11.2 (Pin_2), J7.6 (Pin_6)
- new net: J11.1 (Pin_1), J7.7 (Pin_7)
- new net: J10.5 (Pin_5), J6.1 (Pin_1)
- new net: J10.4 (Pin_4), J6.2 (Pin_2)
